Commit message: [add] add COLLADA data
add base part

File: dhand_description/urdf/base/base.urdf.xacro (robot description, xacro)
@@ -13,10 +13,10 @@
         <material name="blue"/>
         <geometry>
-          <mesh filename="package://dhand_description/meshes/dhand.stl"/>
+          <mesh filename="package://dhand_description/meshes/base/base.dae"/>
         </geometry>
       </visual>
       <collision>
         <geometry>
-          <mesh filename="package://dhand_description/meshes/dhand.stl"/>
+          <mesh filename="package://dhand_description/meshes/base/base.dae"/>
         </geometry>
       </collision>

Commit message: [add] add collada & stl datas
add all collada datas

File: dhand_description/urdf/base/base.urdf.xacro (robot description, xacro)
@@ -13,10 +13,10 @@
         <material name="blue"/>
         <geometry>
-          <mesh filename="package://dhand_description/meshes/base/base.dae"/>
+          <mesh filename="package://dhand_description/meshes/visual/base/base.dae"/>
         </geometry>
       </visual>
       <collision>
         <geometry>
-          <mesh filename="package://dhand_description/meshes/base/base.dae"/>
+          <mesh filename="package://dhand_description/meshes/collision/base/base.stl"/>
         </geometry>
       </collision>
