Commit message: [add] add gazebo element for base part

File: dhand_description/urdf/base/base.gazebo.xacro (robot description, xacro)
@@ -1,8 +1,7 @@
 <?xml version="1.0"?>
 <robot xmlns:xacro="http://ros.org/wiki/xacro">
- <xacro:macro name="dhand_gazebo_v0">
+ <xacro:macro name="dhand_base_gazebo_v0">
 	<gazebo reference="dhand_base_link">
-	  <selfCollide>true</selfCollide>
-	  <material>Gazebo/Blue</material>
+	  <selfCollide>false</selfCollide>
       <mu1 value="0.8" />
       <mu2 value="0.8" />
