Commit message: [add] xacro for urdf
add xacro for urdf.
but gazebo is not yet

File: dhand_description/robots/dhand.urdf.xacro (robot description, xacro)
@@ -1,10 +1,90 @@
 <?xml version="1.0"?>
 <robot name="dhand" xmlns:xacro="http://ros.org/wiki/xacro">
+  <xacro:include filename="$(find dhand_description)/urdf/common.xacro"/>
   <xacro:include filename="$(find dhand_description)/urdf/base/base.urdf.xacro"/>
+  <xacro:include filename="$(find dhand_description)/urdf/finger/finger.urdf.xacro"/>
+  <!-- =============== Inertial Info =============== -->
+  <xacro:property name="finger_base_mass">
+	<mass value="0.04234931"/>
+  </xacro:property>
+  <xacro:property name="finger_middle_mass">
+	<mass value="0.02332939"/>
+  </xacro:property>
+  <xacro:property name="finger_top_mass">
+	<mass value="0.01452790"/>
+  </xacro:property>
+  <xacro:property name="finger_base_inertia">
+	<inertia ixx="0.00003568" ixy="0.00000000" ixz="-0.00001443"
+			 iyy="0.00005208" iyz="0.00000000"
+			 izz="0.00002108" />
+  </xacro:property>
+  <xacro:property name="finger_middle_inertia">
+	<inertia ixx="0.00001418" ixy="0.00000220" ixz="0.00000000"
+			 iyy="0.00000361" iyz="0.00000004"
+			 izz="0.00001530" />
+  </xacro:property>
+  <xacro:property name="finger_top_inertia">
+	<inertia ixx="0.00001842" ixy="0.00000139" ixz="0.00000000"
+			 iyy="0.00000096" iyz="0.00000000"
+			 izz="0.00001830" />
+  </xacro:property>
   <!-- =============== Link & Joint =============== -->
+  <!-- ==== Base ==== -->
   <link name="world"/>
-  <xacro:dhand_v0 parent="world">
+  <xacro:dhand_base_v0 parent="world">
 	<origin xyz="0 0 0" rpy="0 0 0"/>
-  </xacro:dhand_v0>
+  </xacro:dhand_base_v0>
+  <!-- ==== finger base ==== -->
+  <xacro:dhand_fixed_finger_base/>
+  <xacro:dhand_finger_v0 parent="dhand_base_link" prefix="base" side="right">
+  	<origin xyz="0.1865 -0.025964675 -0.01505875" rpy="${90*M_PI/180} 0 ${90*M_PI/180}"/>
+  	<axis xyz="0 0 1"/>
+  	<insert_block name="finger_base_mass"/>
+  	<insert_block name="finger_base_inertia"/>
+  </xacro:dhand_finger_v0>
+  <xacro:dhand_finger_v0 parent="dhand_base_link" prefix="base" side="left">
+  	<origin xyz="0.1865 0.02601464 -0.01494117" rpy="${-90*M_PI/180} 0 ${-90*M_PI/180}"/>
+  	<axis xyz="0 0 1"/>
+  	<insert_block name="finger_base_mass"/>
+  	<insert_block name="finger_base_inertia"/>
+  </xacro:dhand_finger_v0>
+  <!--==== finger middle ====-->
+  <xacro:dhand_finger_v0 parent="dhand_finger_base_middle_link" prefix="middle" side="middle">
+  	<origin xyz="-0.0415 0 0.033" rpy="${90*M_PI/180} 0 0"/>
+  	<axis xyz="0 0 -1"/>
+  	<insert_block name="finger_middle_mass"/>
+  	<insert_block name="finger_middle_inertia"/>
+  </xacro:dhand_finger_v0>
+  <xacro:dhand_finger_v0 parent="dhand_finger_base_right_link" prefix="middle" side="right">
+  	<origin xyz="-0.0415 0 0.033" rpy="${90*M_PI/180} 0 0"/>
+  	<axis xyz="0 0 -1"/>
+  	<insert_block name="finger_middle_mass"/>
+  	<insert_block name="finger_middle_inertia"/>
+  </xacro:dhand_finger_v0>
+  <xacro:dhand_finger_v0 parent="dhand_finger_base_left_link" prefix="middle" side="left">
+  	<origin xyz="-0.0415 0 0.033" rpy="${90*M_PI/180} 0 0"/>
+  	<axis xyz="0 0 -1"/>
+  	<insert_block name="finger_middle_mass"/>
+  	<insert_block name="finger_middle_inertia"/>
+  </xacro:dhand_finger_v0>
+  <!-- ==== finger top ==== -->
+  <xacro:dhand_finger_v0 parent="dhand_finger_middle_middle_link" prefix="top" side="middle">
+  	<origin xyz="0.00976095 0.0434937 0.0" rpy="0 0 0"/>
+  	<axis xyz="0 0 -1"/>
+  	<insert_block name="finger_top_mass"/>
+  	<insert_block name="finger_top_inertia"/>
+  </xacro:dhand_finger_v0>
+   <xacro:dhand_finger_v0 parent="dhand_finger_middle_right_link" prefix="top" side="right">
+  	<origin xyz="0.00976095 0.0434937 0.0" rpy="0 0 0"/>
+  	<axis xyz="0 0 -1"/>
+  	<insert_block name="finger_top_mass"/>
+  	<insert_block name="finger_top_inertia"/>
+   </xacro:dhand_finger_v0>
+    <xacro:dhand_finger_v0 parent="dhand_finger_middle_left_link" prefix="top" side="left">
+  	<origin xyz="0.00976095 0.0434937 0.0" rpy="0 0 0"/>
+  	<axis xyz="0 0 -1"/>
+  	<insert_block name="finger_top_mass"/>
+  	<insert_block name="finger_top_inertia"/>
+  </xacro:dhand_finger_v0>
   <!-- =============== Gazebo =============== -->
   <gazebo>
@@ -12,4 +92,4 @@
     </plugin>
   </gazebo>
-  <xacro:dhand_gazebo_v0/>
+  <xacro:dhand_base_gazebo_v0/>
 </robot>

File: dhand_description/urdf/base/base.urdf.xacro (robot description, xacro)
@@ -3,5 +3,5 @@
   <xacro:include filename="$(find dhand_description)/urdf/materials.xacro"/>
   <xacro:include filename="$(find dhand_description)/urdf/base/base.gazebo.xacro"/>
-  <xacro:macro name="dhand_v0" params="parent *joint_origin">
+  <xacro:macro name="dhand_base_v0" params="parent *joint_origin">
 	<joint name="dhand_base_joint" type="fixed">
 	  <insert_block name="joint_origin"/>
@@ -11,5 +11,4 @@
     <link name="dhand_base_link">
       <visual>
-        <material name="blue"/>
         <geometry>
           <mesh filename="package://dhand_description/meshes/visual/base/base.dae"/>
@@ -18,16 +17,16 @@
       <collision>
         <geometry>
-          <mesh filename="package://dhand_description/meshes/collision/base/base.stl"/>
+          <mesh filename="package://dhand_description/meshes/collision/base.STL"/>
         </geometry>
       </collision>
       <inertial>
-        <mass value="1.57638367963"/>
-        <inertia ixx="1.41435750" ixy="0.00249651" ixz="-0.41662385"
-				 iyy="37.88442518" iyz="0.00518697"
-				 izz="37.62412067" />
+        <mass value="1.22813391"/>
+        <inertia ixx="0.00052834" ixy="0.00000936" ixz="0.00000419"
+				 iyy="0.01395061" iyz="0.00000326"
+				 izz="0.01395381" />
       </inertial>
     </link>
 	<joint name="dhand_palm_joint" type="fixed">
-	  <origin xyz="0.185 0 0"/>
+	  <origin xyz="0.255 0 0"/>
 	  <parent link="dhand_base_link"/>
 	  <child link="dhand_palm_link"/>

Commit message: [add] add adapter part
only urdf.

File: dhand_description/robots/dhand.urdf.xacro (robot description, xacro)
@@ -2,4 +2,5 @@
 <robot name="dhand" xmlns:xacro="http://ros.org/wiki/xacro">
   <xacro:include filename="$(find dhand_description)/urdf/common.xacro"/>
+  <xacro:include filename="$(find dhand_description)/urdf/adapter/adapter.urdf.xacro"/>
   <xacro:include filename="$(find dhand_description)/urdf/base/base.urdf.xacro"/>
   <xacro:include filename="$(find dhand_description)/urdf/finger/finger.urdf.xacro"/>
@@ -30,8 +31,10 @@
   </xacro:property>
   <!-- =============== Link & Joint =============== -->
+  <!-- ==== Adapter ==== -->
+  <link name="world"/>
+  <xacro:dhand_adapter_v0 parent="world"/>
   <!-- ==== Base ==== -->
-  <link name="world"/>
-  <xacro:dhand_base_v0 parent="world">
-	<origin xyz="0 0 0" rpy="0 0 0"/>
+  <xacro:dhand_base_v0 parent="dhand_adapter_link">
+	<origin xyz="0.028 0 0" rpy="0 0 0"/>
   </xacro:dhand_base_v0>
   <!-- ==== finger base ==== -->

File: dhand_description/urdf/base/base.urdf.xacro (robot description, xacro)
@@ -1,5 +1,4 @@
 <?xml version="1.0"?>
 <robot xmlns:xacro="http://ros.org/wiki/xacro">
-  <xacro:include filename="$(find dhand_description)/urdf/materials.xacro"/>
   <xacro:include filename="$(find dhand_description)/urdf/base/base.gazebo.xacro"/>
   <xacro:macro name="dhand_base_v0" params="parent *joint_origin">

Commit message: [modify] add joint limits

File: dhand_description/robots/dhand.urdf.xacro (robot description, xacro)
@@ -41,12 +41,14 @@
   <xacro:dhand_fixed_finger_base/>
   <xacro:dhand_finger_v0 parent="dhand_base_link" prefix="base" side="right">
-  	<origin xyz="0.1865 -0.025964675 -0.01505875" rpy="${90*M_PI/180} 0 ${90*M_PI/180}"/>
+  	<origin xyz="0.1865 -0.025964675 -0.01505875" rpy="${180*M_PI/180} ${-90*M_PI/180} 0"/>
   	<axis xyz="0 0 1"/>
+	<limit effort="10.0" lower="${-120*M_PI/180}" upper="0.0" velocity="10.0"/>
   	<insert_block name="finger_base_mass"/>
   	<insert_block name="finger_base_inertia"/>
   </xacro:dhand_finger_v0>
   <xacro:dhand_finger_v0 parent="dhand_base_link" prefix="base" side="left">
-  	<origin xyz="0.1865 0.02601464 -0.01494117" rpy="${-90*M_PI/180} 0 ${-90*M_PI/180}"/>
+  	<origin xyz="0.1865 0.02601464 -0.01494117" rpy="${-180*M_PI/180} ${-90*M_PI/180} 0"/>
   	<axis xyz="0 0 1"/>
+	<limit effort="10.0" lower="0.0" upper="${120*M_PI/180}" velocity="10.0"/>
   	<insert_block name="finger_base_mass"/>
   	<insert_block name="finger_base_inertia"/>
@@ -56,4 +58,5 @@
   	<origin xyz="-0.0415 0 0.033" rpy="${90*M_PI/180} 0 0"/>
   	<axis xyz="0 0 -1"/>
+	<limit effort="10.0" lower="0.0" upper="0.02" velocity="10.0"/>
   	<insert_block name="finger_middle_mass"/>
   	<insert_block name="finger_middle_inertia"/>
@@ -62,4 +65,5 @@
   	<origin xyz="-0.0415 0 0.033" rpy="${90*M_PI/180} 0 0"/>
   	<axis xyz="0 0 -1"/>
+	<limit effort="10.0" lower="0.0" upper="0.02" velocity="10.0"/>
   	<insert_block name="finger_middle_mass"/>
   	<insert_block name="finger_middle_inertia"/>
@@ -68,4 +72,5 @@
   	<origin xyz="-0.0415 0 0.033" rpy="${90*M_PI/180} 0 0"/>
   	<axis xyz="0 0 -1"/>
+	<limit effort="10.0" lower="0.0" upper="0.02" velocity="10.0"/>
   	<insert_block name="finger_middle_mass"/>
   	<insert_block name="finger_middle_inertia"/>
@@ -75,16 +80,19 @@
   	<origin xyz="0.00976095 0.0434937 0.0" rpy="0 0 0"/>
   	<axis xyz="0 0 -1"/>
+	<limit effort="10.0" lower="0.0" upper="1.40" velocity="10.0"/>
   	<insert_block name="finger_top_mass"/>
   	<insert_block name="finger_top_inertia"/>
   </xacro:dhand_finger_v0>
-   <xacro:dhand_finger_v0 parent="dhand_finger_middle_right_link" prefix="top" side="right">
+  <xacro:dhand_finger_v0 parent="dhand_finger_middle_right_link" prefix="top" side="right">
   	<origin xyz="0.00976095 0.0434937 0.0" rpy="0 0 0"/>
   	<axis xyz="0 0 -1"/>
+	<limit effort="10.0" lower="0.0" upper="1.40" velocity="10.0"/>
   	<insert_block name="finger_top_mass"/>
   	<insert_block name="finger_top_inertia"/>
-   </xacro:dhand_finger_v0>
-    <xacro:dhand_finger_v0 parent="dhand_finger_middle_left_link" prefix="top" side="left">
+  </xacro:dhand_finger_v0>
+  <xacro:dhand_finger_v0 parent="dhand_finger_middle_left_link" prefix="top" side="left">
   	<origin xyz="0.00976095 0.0434937 0.0" rpy="0 0 0"/>
   	<axis xyz="0 0 -1"/>
+	<limit effort="10.0" lower="0.0" upper="1.40" velocity="10.0"/>
   	<insert_block name="finger_top_mass"/>
   	<insert_block name="finger_top_inertia"/>

File: dhand_description/urdf/finger/finger.urdf.xacro (robot description, xacro)
@@ -3,10 +3,12 @@
   <xacro:include filename="$(find dhand_description)/urdf/common.xacro"/>
   <xacro:include filename="$(find dhand_description)/urdf/finger/finger.gazebo.xacro"/>
-  <xacro:macro name="dhand_finger_v0" params="parent prefix side *joint_origin *joint_axis *mass *inertia">
-	<joint name="dhand_finger_${prefix}_${side}_joint" type="continuous">
+  <xacro:macro name="dhand_finger_v0" params="parent prefix side *joint_origin *joint_axis *joint_limit *mass *inertia">
+	<joint name="dhand_finger_${prefix}_${side}_joint" type="revolute">
 	  <insert_block name="joint_origin"/>
 	  <parent link="${parent}"/>
 	  <child link="dhand_finger_${prefix}_${side}_link"/>
 	  <insert_block name="joint_axis"/>
+	  <dynamics damping="0.7" friction="0.7"/>
+	  <insert_block name="joint_limit"/>
 	</joint>
 	<link name="dhand_finger_${prefix}_${side}_link">

Commit message: [modify] change joint origin master -> adapter

File: dhand_description/robots/dhand.urdf.xacro (robot description, xacro)
@@ -3,5 +3,4 @@
   <xacro:include filename="$(find dhand_description)/urdf/common.xacro"/>
   <xacro:include filename="$(find dhand_description)/urdf/adapter/adapter.urdf.xacro"/>
-  <xacro:include filename="$(find dhand_description)/urdf/adapter/adapter.gazebo.xacro"/>
   <xacro:include filename="$(find dhand_description)/urdf/base/base.urdf.xacro"/>
   <xacro:include filename="$(find dhand_description)/urdf/finger/finger.urdf.xacro"/>
@@ -34,5 +33,7 @@
   <!-- ==== Adapter ==== -->
   <link name="world"/>
-  <xacro:dhand_adapter_v0 parent="world"/>
+  <xacro:dhand_adapter_v0 parent="world">
+	<origin xyz="0 0 0.005" rpy="0 ${-M_PI/2} 0"/>
+  </xacro:dhand_adapter_v0>
   <!-- ==== Base ==== -->
   <xacro:dhand_base_v0 parent="dhand_adapter_link">
@@ -127,4 +128,4 @@
   <xacro:dhand_finger_trans_v0 prefix="top" side="middle"/>
   <xacro:dhand_finger_trans_v0 prefix="top" side="right"/>
-  <xacro:dhand_finger_trans_v0 prefix="top" side="lefg"/>
+  <xacro:dhand_finger_trans_v0 prefix="top" side="left"/>
 </robot>

File: dhand_description/urdf/adapter/adapter.urdf.xacro (robot description, xacro)
@@ -1,6 +1,8 @@
 <?xml version="1.0"?>
 <robot xmlns:xacro="http://ros.org/wiki/xacro">
-<xacro:macro name="dhand_adapter_v0" params="parent">
-	<joint name="dhand_adapter_joint" type="fixed">
+<xacro:include filename="$(find dhand_description)/urdf/adapter/adapter.gazebo.xacro"/>
+<xacro:macro name="dhand_adapter_v0" params="parent *joint_origin">
+  <joint name="dhand_adapter_joint" type="fixed">
+	  <insert_block name="joint_origin"/>
 	  <parent link="${parent}"/>
 	  <child link="dhand_adapter_link"/>

Commit message: [modify] modify xacro macro
to make dhand.urdf.xacro simple, modify it.

File: dhand_description/robots/dhand.urdf.xacro (robot description, xacro)
@@ -2,5 +2,4 @@
 <robot name="dhand" xmlns:xacro="http://ros.org/wiki/xacro">
   <xacro:include filename="$(find dhand_description)/urdf/common.xacro"/>
-  <xacro:include filename="$(find dhand_description)/urdf/adapter/adapter.urdf.xacro"/>
   <xacro:include filename="$(find dhand_description)/urdf/base/base.urdf.xacro"/>
   <xacro:include filename="$(find dhand_description)/urdf/finger/finger.urdf.xacro"/>
@@ -31,13 +30,6 @@
   </xacro:property>
   <!-- =============== Link & Joint =============== -->
-  <!-- ==== Adapter ==== -->
-  <link name="world"/>
-  <xacro:dhand_adapter_v0 parent="world">
-	<origin xyz="0 0 0.005" rpy="0 ${-M_PI/2} 0"/>
-  </xacro:dhand_adapter_v0>
   <!-- ==== Base ==== -->
-  <xacro:dhand_base_v0 parent="dhand_adapter_link">
-	<origin xyz="0.028 0 0" rpy="0 0 0"/>
-  </xacro:dhand_base_v0>
+  <xacro:dhand_base_v0 />
   <!-- ==== finger base ==== -->
   <xacro:dhand_fixed_finger_base/>

File: dhand_description/urdf/adapter/adapter.urdf.xacro (robot description, xacro)
@@ -1,11 +1,6 @@
 <?xml version="1.0"?>
 <robot xmlns:xacro="http://ros.org/wiki/xacro">
-<xacro:include filename="$(find dhand_description)/urdf/adapter/adapter.gazebo.xacro"/>
-<xacro:macro name="dhand_adapter_v0" params="parent *joint_origin">
-  <joint name="dhand_adapter_joint" type="fixed">
-	  <insert_block name="joint_origin"/>
-	  <parent link="${parent}"/>
-	  <child link="dhand_adapter_link"/>
-	</joint>
+  <xacro:include filename="$(find dhand_description)/urdf/adapter/adapter.gazebo.xacro"/>
+  <xacro:macro name="dhand_adapter_v0">
     <link name="dhand_adapter_link">
       <visual>
@@ -26,4 +21,4 @@
       </inertial>
     </link>
-</xacro:macro>
+  </xacro:macro>
 </robot>

File: dhand_description/urdf/base/base.urdf.xacro (robot description, xacro)
@@ -2,10 +2,5 @@
 <robot xmlns:xacro="http://ros.org/wiki/xacro">
   <xacro:include filename="$(find dhand_description)/urdf/base/base.gazebo.xacro"/>
-  <xacro:macro name="dhand_base_v0" params="parent *joint_origin">
-	<joint name="dhand_base_joint" type="fixed">
-	  <insert_block name="joint_origin"/>
-	  <parent link="${parent}"/>
-	  <child link="dhand_base_link"/>
-	</joint>
+  <xacro:macro name="dhand_base_v0">
     <link name="dhand_base_link">
       <visual>

Commit message: [fix] fix inertia
put 1e-3 less than that

File: dhand_description/robots/dhand.urdf.xacro (robot description, xacro)
@@ -15,17 +15,17 @@
   </xacro:property>
   <xacro:property name="finger_base_inertia">
-	<inertia ixx="0.00003568" ixy="0.00000000" ixz="-0.00001443"
-			 iyy="0.00005208" iyz="0.00000000"
-			 izz="0.00002108" />
+	<inertia ixx="1e-3" ixy="0.00000000" ixz="-0.00001443"
+			 iyy="1e-3" iyz="0.00000000"
+			 izz="1e-3" />
   </xacro:property>
   <xacro:property name="finger_middle_inertia">
-	<inertia ixx="0.00001418" ixy="0.00000220" ixz="0.00000000"
-			 iyy="0.00000361" iyz="0.00000004"
-			 izz="0.00001530" />
+	<inertia ixx="1e-3" ixy="0.00000220" ixz="0.00000000"
+			 iyy="1e-3" iyz="0.00000004"
+			 izz="1e-3" />
   </xacro:property>
   <xacro:property name="finger_top_inertia">
-	<inertia ixx="0.00001842" ixy="0.00000139" ixz="0.00000000"
-			 iyy="0.00000096" iyz="0.00000000"
-			 izz="0.00001830" />
+	<inertia ixx="1e-3" ixy="0.00000139" ixz="0.00000000"
+			 iyy="1e-3" iyz="0.00000000"
+			 izz="1e-3" />
   </xacro:property>
   <!-- =============== Link & Joint =============== -->

File: dhand_description/urdf/adapter/adapter.urdf.xacro (robot description, xacro)
@@ -16,7 +16,7 @@
       <inertial>
         <mass value="0.09444833"/>
-        <inertia ixx="0.00008749" ixy="0.00000000" ixz="0.00000000"
-				 iyy="0.00008142" iyz="0.00000000"
-				 izz="0.00008142" />
+        <inertia ixx="1e-3" ixy="0.00000000" ixz="0.00000000"
+				 iyy="1e-3" iyz="0.00000000"
+				 izz="1e-3" />
       </inertial>
     </link>

File: dhand_description/urdf/finger/finger.urdf.xacro (robot description, xacro)
@@ -49,7 +49,7 @@
 	  <inertial>
 		<mass value="0.04234931"/>
-		<inertia ixx="0.00003568" ixy="0.00000000" ixz="-0.00001443"
-				 iyy="0.00005208" iyz="0.00000000"
-				 izz="0.00002108" />
+		<inertia ixx="1e-3" ixy="0.00000000" ixz="-0.00001443"
+				 iyy="1e-3" iyz="0.00000000"
+				 izz="1e-3" />
 	  </inertial>
 	</link>

Commit message: [Fix] xacro format to kinetic one

File: dhand_description/robots/dhand.urdf.xacro (robot description, xacro)
@@ -39,6 +39,6 @@
   	<axis xyz="0 0 1"/>
 	<limit effort="10.0" lower="${-120*M_PI/180}" upper="0.0" velocity="10.0"/>
-  	<insert_block name="finger_base_mass"/>
-  	<insert_block name="finger_base_inertia"/>
+  	<xacro:insert_block name="finger_base_mass"/>
+  	<xacro:insert_block name="finger_base_inertia"/>
   </xacro:dhand_finger_v0>
   <xacro:dhand_finger_v0 parent="dhand_base_link" prefix="base" side="left">
@@ -46,6 +46,6 @@
   	<axis xyz="0 0 1"/>
 	<limit effort="10.0" lower="0.0" upper="${120*M_PI/180}" velocity="10.0"/>
-  	<insert_block name="finger_base_mass"/>
-  	<insert_block name="finger_base_inertia"/>
+  	<xacro:insert_block name="finger_base_mass"/>
+  	<xacro:insert_block name="finger_base_inertia"/>
   </xacro:dhand_finger_v0>
   <!--==== finger middle ====-->
@@ -54,6 +54,6 @@
   	<axis xyz="0 0 -1"/>
 	<limit effort="10.0" lower="0.0" upper="0.02" velocity="10.0"/>
-  	<insert_block name="finger_middle_mass"/>
-  	<insert_block name="finger_middle_inertia"/>
+  	<xacro:insert_block name="finger_middle_mass"/>
+  	<xacro:insert_block name="finger_middle_inertia"/>
   </xacro:dhand_finger_v0>
   <xacro:dhand_finger_v0 parent="dhand_finger_base_right_link" prefix="middle" side="right">
@@ -61,6 +61,6 @@
   	<axis xyz="0 0 -1"/>
 	<limit effort="10.0" lower="0.0" upper="0.02" velocity="10.0"/>
-  	<insert_block name="finger_middle_mass"/>
-  	<insert_block name="finger_middle_inertia"/>
+  	<xacro:insert_block name="finger_middle_mass"/>
+  	<xacro:insert_block name="finger_middle_inertia"/>
   </xacro:dhand_finger_v0>
   <xacro:dhand_finger_v0 parent="dhand_finger_base_left_link" prefix="middle" side="left">
@@ -68,6 +68,6 @@
   	<axis xyz="0 0 -1"/>
 	<limit effort="10.0" lower="0.0" upper="0.02" velocity="10.0"/>
-  	<insert_block name="finger_middle_mass"/>
-  	<insert_block name="finger_middle_inertia"/>
+  	<xacro:insert_block name="finger_middle_mass"/>
+  	<xacro:insert_block name="finger_middle_inertia"/>
   </xacro:dhand_finger_v0>
   <!-- ==== finger top ==== -->
@@ -76,6 +76,6 @@
   	<axis xyz="0 0 -1"/>
 	<limit effort="10.0" lower="0.0" upper="1.40" velocity="10.0"/>
-  	<insert_block name="finger_top_mass"/>
-  	<insert_block name="finger_top_inertia"/>
+  	<xacro:insert_block name="finger_top_mass"/>
+  	<xacro:insert_block name="finger_top_inertia"/>
   </xacro:dhand_finger_v0>
   <xacro:dhand_finger_v0 parent="dhand_finger_middle_right_link" prefix="top" side="right">
@@ -83,6 +83,6 @@
   	<axis xyz="0 0 -1"/>
 	<limit effort="10.0" lower="0.0" upper="1.40" velocity="10.0"/>
-  	<insert_block name="finger_top_mass"/>
-  	<insert_block name="finger_top_inertia"/>
+  	<xacro:insert_block name="finger_top_mass"/>
+  	<xacro:insert_block name="finger_top_inertia"/>
   </xacro:dhand_finger_v0>
   <xacro:dhand_finger_v0 parent="dhand_finger_middle_left_link" prefix="top" side="left">
@@ -90,6 +90,6 @@
   	<axis xyz="0 0 -1"/>
 	<limit effort="10.0" lower="0.0" upper="1.40" velocity="10.0"/>
-  	<insert_block name="finger_top_mass"/>
-  	<insert_block name="finger_top_inertia"/>
+  	<xacro:insert_block name="finger_top_mass"/>
+  	<xacro:insert_block name="finger_top_inertia"/>
   </xacro:dhand_finger_v0>
   <!-- =============== Gazebo =============== -->

File: dhand_description/urdf/common.xacro (robot description, xacro)
@@ -1,4 +1,4 @@
 <?xml version="1.0"?>
 <robot xmlns:xacro="http://ros.org/wiki/xacro">
-  <property name="M_PI" value="3.14159274"/>
+  <xacro:property name="M_PI" value="3.14159274"/>
 </robot>

File: dhand_description/urdf/finger/finger.urdf.xacro (robot description, xacro)
@@ -6,10 +6,10 @@
   <xacro:macro name="dhand_finger_v0" params="parent prefix side *joint_origin *joint_axis *joint_limit *mass *inertia">
 	<joint name="dhand_finger_${prefix}_${side}_joint" type="revolute">
-	  <insert_block name="joint_origin"/>
+	  <xacro:insert_block name="joint_origin"/>
 	  <parent link="${parent}"/>
 	  <child link="dhand_finger_${prefix}_${side}_link"/>
-	  <insert_block name="joint_axis"/>
+	  <xacro:insert_block name="joint_axis"/>
 	  <dynamics damping="0.7" friction="0.7"/>
-	  <insert_block name="joint_limit"/>
+	  <xacro:insert_block name="joint_limit"/>
 	</joint>
 	<link name="dhand_finger_${prefix}_${side}_link">
@@ -25,6 +25,6 @@
 	  </collision>
 	  <inertial>
-		<insert_block name="mass"/>
-	  	<insert_block name="inertia"/>
+		<xacro:insert_block name="mass"/>
+	  	<xacro:insert_block name="inertia"/>
 	  </inertial>
 	</link>
